Commit message: 0930

File: models/indy7_coarse/indy7.urdf (robot description, URDF)
Before this commit: robot indy7, 9 links, 8 joints
Links:
- added link base_link
Joints:
- added joint base_joint: type fixed, parent base_link, child link0, origin xyz=0 0 0 rpy=0 0 0, axis 0 0 1, limit lower=-3.05432619099 upper=3.05432619099 effort=10 velocity=1
- joint world_fixed: child link0 -> base_link; origin xyz=1 1 0 rpy=0 0 0 -> xyz=1.5 1.5 0 rpy=0 0 0

File: models/indy7_collision_coarse/indy7.urdf (robot description, URDF)
Before this commit: robot indy7_collision, 9 links, 8 joints
Joints:
- joint world_fixed: origin xyz=1 1 0 rpy=0 0 0 -> xyz=1.5 1.5 0 rpy=0 0 0
